File: boards/bandoneon/bandoneon.kicad_pcb (KiCad board)
At the start: 2 copper layers, 405 x 100 mm, 84 parts, among them J1 2D JOYSTICK, J3 JST XH-3A, U1 Feather M4 Express, U10 MCP3008, U2 MCP3008, U3 MCP3008, U4 MCP3008, U5 MCP3008, U6 MCP3008, U7 MCP3008, U8 MCP3008, U9 MCP3008

Commit message: Printing carter attempt.
Parts:
- added REF**: MountingHole_2.1mm, MountingHole:MountingHole_2.1mm, F.Cu at (239.1, 261.6)
- added REF**: MountingHole_2.1mm, MountingHole:MountingHole_2.1mm, F.Cu at (371.8, 261.8)
- moved J3 38.1 mm to (263.0, 123.0)
- moved H38 33.2 mm to (180.5, 126.5), turned to 33 degrees
- moved H20 32.0 mm to (203.8, 128.7), turned to 33 degrees
- moved H35 31.5 mm to (169.5, 137.4), turned to 33 degrees
- moved U1 31.3 mm to (290.0, 127.5)
- moved H30 31.2 mm to (225.6, 132.4), turned to -57 degrees
- moved H7 30.9 mm to (325.3, 166.2), turned to -33 degrees
- moved H44 30.8 mm to (455.0, 145.5), turned to 57 degrees
- moved H8 30.7 mm to (247.9, 138.4), turned to -57 degrees
- moved H70 30.7 mm to (420.2, 136.9), turned to 57 degrees
- moved H21 30.4 mm to (191.6, 137.7), turned to 33 degrees
- moved H65 30.3 mm to (394.7, 140.1), turned to 57 degrees
- moved H36 29.9 mm to (159.4, 149.6), turned to 33 degrees
- moved H52 29.7 mm to (371.9, 146.2), turned to 57 degrees
- moved H61 29.5 mm to (347.7, 154.7), turned to 57 degrees
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Other:
- board size 405 x 100 mm -> 370 x 150 mm
