File: boards/bandoneon/bandoneon.kicad_pcb (KiCad board)
At the start: 2 copper layers, 384.9 x 143.8 mm, 122 parts, among them J1 2D JOYSTICK, J4 AudioJack3, J5 AudioJack3, J6 JST XH-3A, J7 JST XH-3A, U1 Feather M4 Express, U10 MCP3008, U11 SRV05-4, U12 SRV05-4, U13 SRV05-4, U2 MCP3008, U3 MCP3008, U4 MCP3008, U5 MCP3008, U6 MCP3008, U7 MCP3008, U8 MCP3008, U9 MCP3008

Commit message: Before setting up the bom + pick and place
Parts:
- moved U12 1.93 mm to (296.2, 200.2)
Routing:
- net GND: track 552.3 -> 565.2 mm, vias 88 -> 91
- net /VBUS: track 9.63 -> 7.69 mm
- net /CLK: track 396.3 -> 398.1 mm
- net /EXPR_PED: track 135.1 -> 136.3 mm
