File: boards/bandoneon/bandoneon.kicad_pcb (KiCad board)
At the start: 2 copper layers, 384.9 x 143.8 mm, 122 parts, among them J1 2D JOYSTICK, J4 AudioJack3, J5 AudioJack3, J6 JST XH-3A, J7 JST XH-3A, U1 Feather M4 Express, U10 MCP3008, U11 SRV05-4, U12 SRV05-4, U13 SRV05-4, U2 MCP3008, U3 MCP3008, U4 MCP3008, U5 MCP3008, U6 MCP3008, U7 MCP3008, U8 MCP3008, U9 MCP3008

Commit message: Annotate TRS.
Other:
- board text added: "expr"
- board text added: "sus"
Changed lines of the file:
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@@
     )
+  )
+  (gr_text "sus" (at 338.7598 146.9898) (layer "F.Cu")
+    (effects (font (size 1.5 1.5) (thickness 0.3) bold) (justify left bottom))
+  )
+  (gr_text "expr" (at 362.839 147.1168) (layer "F.Cu")
+    (effects (font (size 1.5 1.5) (thickness 0.3) bold) (justify left bottom))
   )
   (gr_text "https://github.com/piwicode/bandoneon" (at 394.716 251.968 12) (layer "F.SilkS")
