File: boards/bandoneon/_autosave-bandoneon.kicad_sch (KiCad schematic)
At the start: 11 parts, among them J1 AudioJack3, J2 AudioJack3, J3 JST XH-3A, J4 JST XH-3A, J6 2D JOYSTICK, J6 JST XH-3A, J8 JST XH-3A, U10 Feather M4 Express

Commit message: Ready for routing
Parts:
- renumbered J6 to J1, J6 to J2, J8 to J3, J1 to J4, J2 to J5, J3 to J6, J4 to J7, RV4 to RV1, RV5 to RV2, U10 to U1
