File: boards/bandoneon/bandoneon_auto.kicad_pcb (KiCad board)
At the start: 2 copper layers, 384.9 x 143.8 mm, 111 parts, among them J1 2D JOYSTICK, J4 AudioJack3, J5 AudioJack3, J6 JST XH-3A, J7 JST XH-3A, U1 Feather M4 Express, U10 MCP3008, U2 MCP3008, U3 MCP3008, U4 MCP3008, U5 MCP3008, U6 MCP3008, U7 MCP3008, U8 MCP3008, U9 MCP3008

Commit message: Manual routing
Parts:
- removed the MH13 at (370.2, 213.4)
- removed the MH14 at (283.2, 234.9)
- added J9: JST XH-3A, Connector_JST:JST_XH_B3B-XH-A_1x03_P2.50mm_Vertical, B.Cu at (278.5, 124.0)
- added MH15: MountingHole_3.2mm_M3_large, Library:MountingHole_3.2mm_M3_large, F.Cu at (251.5, 225.5)
- moved U3 73.7 mm to (275.0, 154.5), turned to 0 degrees
- moved H58 62.8 mm to (338.3, 214.3)
- moved H19 53.7 mm to (191.6, 137.6)
- moved H10 53.5 mm to (256.2, 151.0), turned to -57 degrees
- moved H31 52.6 mm to (188.8, 187.7)
- moved H30 51.3 mm to (199.7, 176.4), turned to 33 degrees
- moved U2 45.2 mm to (281.5, 185.8), turned to 0 degrees
- moved H46 40.2 mm to (443.2, 145.3)
- moved H47 40.2 mm to (443.2, 185.5)
- moved H3 39.8 mm to (228.9, 197.1), turned to 33 degrees
- moved H9 39.7 mm to (234.0, 145.0), turned to -57 degrees
- moved H68 38.4 mm to (421.8, 185.7)
- moved H62 38.3 mm to (357.8, 154.6)
- moved H21 38.2 mm to (179.8, 173.9)
- moved H7 37.7 mm to (274.4, 200.7), turned to 54 degrees
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Connections:
- J6 pad 3: +3.3V -> /3V3
- J7 pad 3: +3.3V -> /3V3
- U1 pad 10: /G7/MISO -> /G4/MISO
- U1 pad 11: /G10/MISO -> /G3/MISO
- U1 pad 14: /SUS_PED -> /JOY_BT
- U1 pad 15: /JOY_BT -> /SUS_PED
- U1 pad 16: /G6/MISO -> /G2/MISO
- U1 pad 17: /G9/MISO -> /G5/MISO
- U1 pad 18: /G5/MISO -> /G1/MISO
- U1 pad 19: /G3/MISO -> /G6/MISO
- U1 pad 20: /G4/MISO -> /G7/MISO
- U1 pad 21: /G2/MISO -> /G10/MISO
- U1 pad 22: /G1/MISO -> /G9/MISO
- U2 pad 1: unconnected-(U2-CH0-Pad1) -> Net-(J9-Pin_2)
Routing:
- net GND: track 53.2 -> 1979.1 mm, vias 0 -> 28
- net +3.3V: track 1969.2 -> 1871.9 mm, vias 0 -> 14
- net Net-(J9-Pin_2): track 0.00 -> 61.9 mm, vias 0 -> 1
- net Net-(H19-OUT): track 12.5 -> 70.6 mm, vias 0 -> 2
- net /MOSI: track 401.4 -> 452.2 mm, vias 9 -> 8
- net Net-(H21-OUT): track 76.2 -> 26.1 mm, vias 0 -> 2
- net Net-(H30-OUT): track 85.8 -> 35.9 mm, vias 0 -> 2
- net Net-(H1-OUT): track 113.1 -> 64.9 mm
- net /CLK: track 390.0 -> 437.9 mm, vias 9 -> 10
- net Net-(H7-OUT): track 65.2 -> 19.5 mm, vias 0 -> 2
- net Net-(H46-OUT): track 26.1 -> 68.9 mm, vias 0 -> 2
- net Net-(H3-OUT): track 14.9 -> 56.9 mm, vias 0 -> 2
- net /CS: track 409.6 -> 450.4 mm, vias 9 -> 6
- net Net-(H11-OUT): track 73.8 -> 33.6 mm
- net Net-(H68-OUT): track 69.0 -> 28.9 mm, vias 0 -> 2
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