File: boards/bandoneon/grape_alt.kicad_sch (KiCad schematic)
At the start: 9 parts, among them U2 MCP3008

Commit message: Gerber and bom export
Parts:
- C9: LCSC Part (none) -> C52923
- H1, H2, H3, H4, H5, H6, H7: value ~ -> SS39ET; footprint Library:SS39ET -> Library:SOT-23_SS39ET; LCSC Part (none) -> C126669
- U2: footprint Library:MCP3008T-I_SL -> Library:SOIC-16_MCP3008T-I_SL; LCSC C1520159 -> (none); LCSC Part (none) -> C1520159
Changed lines of the file:
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@@
       (effects (font (size 1.27 1.27)))
     )
-    (property "Value" "~" (at 40.64 78.74 0)
-      (effects (font (size 1.27 1.27)))
-    )
-    (property "Footprint" "Library:SS39ET" (at 40.64 78.74 0)
-      (effects (font (size 1.27 1.27)) hide)
-    )
-    (property "Datasheet" "" (at 40.64 78.74 0)
+    (property "Value" "SS39ET" (at 35.56 80.01 90)
+      (effects (font (size 1.27 1.27)))
+    )
+    (property "Footprint" "Library:SOT-23_SS39ET" (at 40.64 85.09 0)
+      (effects (font (size 1.27 1.27)) hide)
+    )
+    (property "Datasheet" "https://jlcpcb.com/partdetail/Honeywell-SS39ET/C126669" (at 40.64 88.9 0)
+      (effects (font (size 1.27 1.27)) hide)
+    )
+    (property "LCSC Part" "C126669" (at 39.37 87.122 0)
       (effects (font (size 1.27 1.27)) hide)
     )
@@
       (effects (font (size 1.27 1.27)))
     )
-    (property "Value" "~" (at 40.64 53.34 0)
-      (effects (font (size 1.27 1.27)))
-    )
-    (property "Footprint" "Library:SS39ET" (at 40.64 53.34 0)
-      (effects (font (size 1.27 1.27)) hide)
-    )
-    (property "Datasheet" "" (at 40.64 53.34 0)
+    (property "Value" "SS39ET" (at 35.56 54.61 90)
+      (effects (font (size 1.27 1.27)))
+    )
+    (property "Footprint" "Library:SOT-23_SS39ET" (at 40.64 59.69 0)
+      (effects (font (size 1.27 1.27)) hide)
+    )
+    (property "Datasheet" "https://jlcpcb.com/partdetail/Honeywell-SS39ET/C126669" (at 40.64 63.5 0)
+      (effects (font (size 1.27 1.27)) hide)
+    )
+    (property "LCSC Part" "C126669" (at 39.37 61.722 0)
       (effects (font (size 1.27 1.27)) hide)
     )
@@
       (effects (font (size 1.27 1.27)))
     )
-    (property "Value" "~" (at 40.64 116.84 0)
-      (effects (font (size 1.27 1.27)))
-    )
-    (property "Footprint" "Library:SS39ET" (at 40.64 116.84 0)
-      (effects (font (size 1.27 1.27)) hide)
-    )
-    (property "Datasheet" "" (at 40.64 116.84 0)
+    (property "Value" "SS39ET" (at 35.56 118.11 90)
+      (effects (font (size 1.27 1.27)))
+    )
+    (property "Footprint" "Library:SOT-23_SS39ET" (at 40.64 123.19 0)
+      (effects (font (size 1.27 1.27)) hide)
+    )
+    (property "Datasheet" "https://jlcpcb.com/partdetail/Honeywell-SS39ET/C126669" (at 40.64 127 0)
+      (effects (font (size 1.27 1.27)) hide)
+    )
+    (property "LCSC Part" "C126669" (at 39.37 125.222 0)
       (effects (font (size 1.27 1.27)) hide)
     )
@@
       (effects (font (size 1.27 1.27)) hide)
     )
-    (property "Datasheet" "~" (at 125.095 67.31 0)
+    (property "Datasheet" "https://jlcpcb.com/partdetail/53938-CL05A105KA5NQNC/C52923" (at 125.095 67.31 0)
+      (effects (font (size 1.27 1.27)) hide)
+    )
+    (property "LCSC Part" "C52923" (at 125.095 67.31 0)
       (effects (font (size 1.27 1.27)) hide)
     )
@@
     (in_bom yes) (on_board yes) (dnp no)
     (property "Reference" "H1" (at 39.37 35.56 0)
-      (effects (font (size 1.27 1.27)) hide)
-    )
-    (property "Value" "~" (at 40.64 40.64 0)
-      (effects (font (size 1.27 1.27)))
-    )
-    (property "Footprint" "Library:SS39ET" (at 40.64 40.64 0)
-      (effects (font (size 1.27 1.27)) hide)
-    )
-    (property "Datasheet" "" (at 40.64 40.64 0)
+      (effects (font (size 1.27 1.27)))
+    )
+    (property "Value" "SS39ET" (at 35.56 41.91 90)
+      (effects (font (size 1.27 1.27)))
+    )
+    (property "Footprint" "Library:SOT-23_SS39ET" (at 40.64 46.99 0)
+      (effects (font (size 1.27 1.27)) hide)
+    )
+    (property "Datasheet" "https://jlcpcb.com/partdetail/Honeywell-SS39ET/C126669" (at 40.64 50.8 0)
+      (effects (font (size 1.27 1.27)) hide)
+    )
+    (property "LCSC Part" "C126669" (at 39.37 49.022 0)
       (effects (font (size 1.27 1.27)) hide)
     )
@@
       (effects (font (size 1.27 1.27)))
     )
-    (property "Value" "~" (at 40.64 66.04 0)
-      (effects (font (size 1.27 1.27)))
-    )
-    (property "Footprint" "Library:SS39ET" (at 40.64 66.04 0)
-      (effects (font (size 1.27 1.27)) hide)
-    )
-    (property "Datasheet" "" (at 40.64 66.04 0)
+    (property "Value" "SS39ET" (at 35.56 67.31 90)
+      (effects (font (size 1.27 1.27)))
+    )
+    (property "Footprint" "Library:SOT-23_SS39ET" (at 40.64 72.39 0)
+      (effects (font (size 1.27 1.27)) hide)
+    )
+    (property "Datasheet" "https://jlcpcb.com/partdetail/Honeywell-SS39ET/C126669" (at 40.64 76.2 0)
+      (effects (font (size 1.27 1.27)) hide)
+    )
+    (property "LCSC Part" "C126669" (at 39.37 74.422 0)
       (effects (font (size 1.27 1.27)) hide)
     )
@@
       (effects (font (size 1.27 1.27)) (justify left))
     )
-    (property "Footprint" "Library:MCP3008T-I_SL" (at 90.17 64.77 0)
+    (property "Footprint" "Library:SOIC-16_MCP3008T-I_SL" (at 90.17 64.77 0)
       (effects (font (size 1.27 1.27)) hide)
     )
@@
       (effects (font (size 1.27 1.27)) hide)
     )
-    (property "LCSC" "C1520159" (at 87.63 67.31 0)
+    (property "LCSC Part" "C1520159" (at 87.63 67.31 0)
       (effects (font (size 1.27 1.27)) hide)
     )
@@
       (effects (font (size 1.27 1.27)))
     )
-    (property "Value" "~" (at 40.64 91.44 0)
-      (effects (font (size 1.27 1.27)))
-    )
-    (property "Footprint" "Library:SS39ET" (at 40.64 91.44 0)
-      (effects (font (size 1.27 1.27)) hide)
-    )
-    (property "Datasheet" "" (at 40.64 91.44 0)
+    (property "Value" "SS39ET" (at 35.56 92.71 90)
+      (effects (font (size 1.27 1.27)))
+    )
+    (property "Footprint" "Library:SOT-23_SS39ET" (at 40.64 97.79 0)
+      (effects (font (size 1.27 1.27)) hide)
+    )
+    (property "Datasheet" "https://jlcpcb.com/partdetail/Honeywell-SS39ET/C126669" (at 40.64 101.6 0)
+      (effects (font (size 1.27 1.27)) hide)
+    )
+    (property "LCSC Part" "C126669" (at 39.37 99.822 0)
       (effects (font (size 1.27 1.27)) hide)
     )
@@
       (effects (font (size 1.27 1.27)))
     )
-    (property "Value" "~" (at 40.64 104.14 0)
-      (effects (font (size 1.27 1.27)))
-    )
-    (property "Footprint" "Library:SS39ET" (at 40.64 104.14 0)
-      (effects (font (size 1.27 1.27)) hide)
-    )
-    (property "Datasheet" "" (at 40.64 104.14 0)
-      (effects (font (size 1.27 1.27)) hide)
-    )
+    (property "Value" "SS39ET" (at 35.56 105.41 90)
+      (effects (font (size 1.27 1.27)))
+    )
+    (property "Footprint" "Library:SOT-23_SS39ET" (at 40.64 110.49 0)
+      (effects (font (size 1.27 1.27)) hide)
+    )
+    (property "Datasheet" "https://jlcpcb.com/partdetail/Honeywell-SS39ET/C126669" (at 40.64 114.3 0)
+      (effects (font (size 1.27 1.27)) hide)
+    )
+    (property "LCSC Part" "C126669" (at 39.37 112.522 0)
+      (effects (font (size 1.27 1.27)) hide)
+    )
